File: Smallpaw.kicad_pcb (KiCad board)
At the start: 2 copper layers, 328.6 x 83.3 mm, 145 parts, among them J1 USB_mini_micro_B, K1 KEYSW, K10 KEYSW, K11 KEYSW, K12 KEYSW, K13 KEYSW, K14 KEYSW, K15 KEYSW, K16 KEYSW, K17 KEYSW, K17.2 KEYSW, K18 KEYSW, K19 KEYSW, K2 KEYSW, K20 KEYSW, K21 KEYSW, K22 KEYSW, K23 KEYSW, K24 KEYSW, K25 KEYSW, K26 KEYSW, K27 KEYSW, K28 KEYSW, K29 KEYSW, K3 KEYSW, K30 KEYSW, K31 KEYSW, K32 KEYSW, K33 KEYSW, K34 KEYSW, K35 KEYSW, K36 KEYSW, K37 KEYSW, K38 KEYSW, K39 KEYSW, K4 KEYSW, K40 KEYSW, K41 KEYSW, K42 KEYSW, K43 KEYSW, K44 KEYSW, K45 KEYSW, K46 KEYSW, K47 KEYSW, K48 KEYSW, K48.2 KEYSW, K49 KEYSW, K5 KEYSW, K50 KEYSW, K51 KEYSW, K52 KEYSW, K53 KEYSW, K54 KEYSW, K55 KEYSW, K56 KEYSW, K57 KEYSW, K58 KEYSW, K59 KEYSW, K6 KEYSW, K60 KEYSW, K61 KEYSW, K62 KEYSW, K63 KEYSW, K7 KEYSW, K8 KEYSW, K9 KEYSW, SW1 SW_PUSH, U1 ATMEGA32U4, X1 XTAL_GND

Commit message: jaja blabla or ckck ckck
Parts:
- removed G***: LOGO, SPSilks:smallpaw_f
- moved C7 2.35 mm to (123.5, 74.3)
Connections:
- U1 pad 31: Net-(U1-Pad31) -> /R6
- U1 pad 32: Net-(U1-Pad32) -> /R5
- U1 pad 36: Net-(U1-Pad36) -> /R4
- U1 pad 37: Net-(U1-Pad37) -> /C1
- U1 pad 38: Net-(U1-Pad38) -> /C0
- U1 pad 39: Net-(U1-Pad39) -> /R0
- U1 pad 40: Net-(U1-Pad40) -> /R1
- U1 pad 41: Net-(U1-Pad41) -> /R3
- U1 pad 42: Net-(U1-Pad42) -> /R2
Routing:
- net /R3: track 260.0 -> 291.3 mm, vias 4 -> 6
- net /R6: track 304.7 -> 332.2 mm, vias 0 -> 2
- net /R5: track 274.2 -> 285.8 mm, vias 2 -> 0
- net /R2: track 291.4 -> 301.1 mm, vias 4 -> 6
- net /R4: track 299.1 -> 303.2 mm, vias 2 -> 3
- net VCC: track 95.2 -> 92.7 mm

Commit message: routed rows/columns
Parts:
- added G***: LOGO, SPSilks:smallpaw_f, F.Cu at (219.2, 80.7)
- K17.2: footprint MX_Alps_Hybrid:MX-2U-ReversedStabilizers-NoLED -> MX_Alps_Hybrid:MX-2U-NoLED
- moved D63 21.8 mm to (352.4, 108.9)
- moved C5 2.49 mm to (135.6, 91.0), turned to 270 degrees
- moved C3 1.18 mm to (127.1, 91.5)
Connections:
- U1 pad 11: Net-(U1-Pad11) -> /R0
- U1 pad 20: /R4 -> Net-(U1-Pad20)
- U1 pad 21: Net-(U1-Pad21) -> /C2
- U1 pad 22: /C2 -> /C7
- U1 pad 25: Net-(U1-Pad25) -> /C6
- U1 pad 26: Net-(U1-Pad26) -> /C5
- U1 pad 27: Net-(U1-Pad27) -> /C4
- U1 pad 28: Net-(U1-Pad28) -> /C3
- U1 pad 29: Net-(U1-Pad29) -> /R6
- U1 pad 30: Net-(U1-Pad30) -> /R7
- U1 pad 31: /R6 -> /C0
- U1 pad 36: /R4 -> /C1
- U1 pad 37: /C1 -> Net-(U1-Pad37)
- U1 pad 38: /C0 -> Net-(U1-Pad38)
- U1 pad 39: /R0 -> /R4
Routing:
- net /C7: track 154.2 -> 403.9 mm
- net /C6: track 165.8 -> 350.6 mm, vias 0 -> 1
- net /C5: track 160.0 -> 303.3 mm, vias 0 -> 1
- net /C4: track 127.2 -> 233.1 mm, vias 0 -> 1
- net /R1: track 264.8 -> 336.0 mm, vias 2 -> 4
- net /C0: track 136.6 -> 204.2 mm
- net /C3: track 148.4 -> 210.9 mm, vias 0 -> 1
- net /R6: track 332.2 -> 362.8 mm
- net /R0: track 310.9 -> 333.1 mm
- net GND: track 49.8 -> 65.7 mm, vias 3 -> 7
- net Net-(D63-Pad2): track 6.89 -> 18.4 mm
- net /C1: track 136.7 -> 148.2 mm
- net VCC: track 92.7 -> 94.6 mm
- net /R7: track 291.2 -> 293.1 mm, vias 2 -> 0
- net /C2: track 153.9 -> 155.4 mm
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Other:
- board size 328.6 x 83.3 mm -> 322.6 x 78.1 mm

Commit message: miniusb
Parts:
- removed X1: XTAL_GND, keyboard_parts:FA-238
- added F1: 500 mA, keebio-parts:Fuse_0805, B.Cu at (149.0, 55.0)
- added Y1: Crystal_GND24_Small, Crystals:Crystal_SMD_SeikoEpson_FA238-4pin_3.2x2.5mm, B.Cu at (146.2, 80.1)
- J1: footprint keyboard_parts:USB_microB -> keebio-parts:USB-Mini-B_ LCSC-C46398
- SW1: footprint Button_Switch_SMD:SW_SPST_TL3342 -> Buttons_Switches_SMD:SW_SPST_SKQG
- moved J1 4.95 mm to (147.6, 47.2)
- moved C4 0.85 mm to (121.6, 77.1)
Connections:
- C3 pad 1: VCC -> +5V
- C4 pad 1: VCC -> +5V
- C5 pad 1: VCC -> +5V
- C6 pad 1: VCC -> +5V
- C7 pad 1: VCC -> +5V
- R1 pad 2: VCC -> +5V
- U1 pad 14: VCC -> +5V
- U1 pad 2: VCC -> +5V
- U1 pad 24: VCC -> +5V
- U1 pad 34: VCC -> +5V
- U1 pad 44: VCC -> +5V
- U1 pad 7: VCC -> +5V
Routing:
- net +5V: track 0.00 -> 84.9 mm
- net VCC: track 94.6 -> 20.1 mm
- net GND: track 65.7 -> 72.3 mm, vias 7 -> 3
- net Net-(J1-Pad2): track 36.0 -> 39.6 mm
- net /R1: track 336.0 -> 332.8 mm, vias 4 -> 2
- net Net-(J1-Pad3): track 32.3 -> 29.4 mm
- net /R2: track 301.1 -> 302.4 mm, vias 6 -> 4
- net /R3: track 292.5 -> 292.0 mm
