File: Smallpaw.sch (KiCad schematic (older format))
At the start: 144 parts, among them J1 USB_mini_micro_B, K1 KEYSW, K10 KEYSW, K11 KEYSW, K12 KEYSW, K13 KEYSW, K14 KEYSW, K15 KEYSW, K16 KEYSW, K17 KEYSW, K17.2 KEYSW, K18 KEYSW, K19 KEYSW, K2 KEYSW, K20 KEYSW, K21 KEYSW, K22 KEYSW, K23 KEYSW, K24 KEYSW, K25 KEYSW, K26 KEYSW, K27 KEYSW, K28 KEYSW, K29 KEYSW, K3 KEYSW, K30 KEYSW, K31 KEYSW, K32 KEYSW, K33 KEYSW, K34 KEYSW, K35 KEYSW, K36 KEYSW, K37 KEYSW, K38 KEYSW, K39 KEYSW, K4 KEYSW, K40 KEYSW, K41 KEYSW, K42 KEYSW, K43 KEYSW, K44 KEYSW, K45 KEYSW, K46 KEYSW, K47 KEYSW, K48 KEYSW, K48.2 KEYSW, K49 KEYSW, K5 KEYSW, K50 KEYSW, K51 KEYSW, K52 KEYSW, K53 KEYSW, K54 KEYSW, K55 KEYSW, K56 KEYSW, K57 KEYSW, K58 KEYSW, K59 KEYSW, K6 KEYSW, K60 KEYSW, K61 KEYSW, K62 KEYSW, K63 KEYSW, K7 KEYSW, K8 KEYSW, K9 KEYSW, SW1 SW_PUSH, U1 ATMEGA32U4, X1 XTAL_GND

Commit message: jaja blabla or ckck ckck
Changed lines of the file:
@@
 EESchema Schematic File Version 4
 LIBS:Smallpaw-cache
-LIBS:Voyager65-cache
 EELAYER 26 0
 EELAYER END
@@
 Text Label 4400 3050 2    50   ~ 0
 R4
+Text Label 6550 1750 0    50   ~ 0
+C0
+Text Label 6550 1850 0    50   ~ 0
+C1
+Text Label 6550 1650 0    50   ~ 0
+R0
+Text Label 6550 1550 0    50   ~ 0
+R1
+Text Label 6550 1350 0    50   ~ 0
+R2
+Text Label 6550 1450 0    50   ~ 0
+R3
+Text Label 6550 1950 0    50   ~ 0
+R4
+Text Label 6550 2450 0    50   ~ 0
+R6
+Text Label 6550 2350 0    50   ~ 0
+R5
 $EndSCHEMATC

Commit message: routed rows/columns
Parts:
- J1: symbol keyboard_parts:USB_mini_micro_B -> Smallpaw-rescue:USB_mini_micro_B-keyboard_parts
- K1, K10, K11, K12, K13, K14, K15, K16, K17, K18, K19, K2, K20, K21, K22, K23, K24, K25, K26, K27, K28, K29, K3, K30, K31, K32, K33, K34, K35, K36, K37, K38, K39, K4, K40, K41, K42, K43, K44, K45, K46, K47, K48, K48.2, K49, K5, K50, K51, K52, K53, K54, K55, K56, K57, K58, K59, K6, K60, K61, K62, K63, K7, K8, K9: symbol keyboard_parts:KEYSW -> Smallpaw-rescue:KEYSW-keyboard_parts
- K17.2: footprint MX_Alps_Hybrid:MX-2U-ReversedStabilizers-NoLED -> MX_Alps_Hybrid:MX-2U-NoLED; symbol keyboard_parts:KEYSW -> Smallpaw-rescue:KEYSW-keyboard_parts
- SW1: symbol keyboard_parts:SW_PUSH -> Smallpaw-rescue:SW_PUSH-keyboard_parts
- U1: symbol keyboard_parts:ATMEGA32U4 -> Smallpaw-rescue:ATMEGA32U4-keyboard_parts
- X1: symbol keyboard_parts:XTAL_GND -> Smallpaw-rescue:XTAL_GND-keyboard_parts
Connections:
- no-connect marks 1 -> 17

Commit message: miniusb
Parts:
- removed X1: XTAL_GND, keyboard_parts:FA-238, symbol Smallpaw-rescue:XTAL_GND-keyboard_parts
- added F1: 500 mA, keebio-parts:Fuse_0805, symbol Device:Polyfuse_Small
- added Y1: Crystal_GND24_Small, Crystals:Crystal_SMD_SeikoEpson_FA238-4pin_3.2x2.5mm, symbol Device:Crystal_GND24_Small
- J1: footprint keyboard_parts:USB_microB -> keebio-parts:USB-Mini-B_ LCSC-C46398
- SW1: footprint Button_Switch_SMD:SW_SPST_TL3342 -> Buttons_Switches_SMD:SW_SPST_SKQG
Connections:
- net GND: now also Y1.2, Y1.4
- net VCC: now also F1.2; no longer C3.1, C4.1, C5.1, C6.1, C7.1, R1.2, U1.14 (VCC), U1.2 (UVcc), U1.24 (AVCC), U1.34 (VCC), U1.44 (AVCC), U1.7 (VBus)
- net at C1.2, U1.16 (XTAL1): now also Y1.1
- net at C2.2, U1.17 (XTAL2): now also Y1.3
- new net +5V: C3.1, C4.1, C5.1, C6.1, C7.1, F1.1, R1.2, U1.14 (VCC), U1.2 (UVcc), U1.24 (AVCC), U1.34 (VCC), U1.44 (AVCC), U1.7 (VBus)
Other:
- moved on the sheet: C1, C2
Changed lines of the file:
@@
 L Device:C_Small C1
 U 1 1 5B8472FB
-P 3000 3100
-F 0 "C1" H 2908 3054 50  0000 R CNN
-F 1 "22p" H 2908 3145 50  0000 R CNN
-F 2 "Capacitor_SMD:C_0805_2012Metric_Pad1.15x1.40mm_HandSolder" H 3000 3100 50  0001 C CNN
-F 3 "~" H 3000 3100 50  0001 C CNN
-	1    3000 3100
+P 3000 2950
+F 0 "C1" H 2908 2904 50  0000 R CNN
+F 1 "22p" H 2908 2995 50  0000 R CNN
+F 2 "Capacitor_SMD:C_0805_2012Metric_Pad1.15x1.40mm_HandSolder" H 3000 2950 50  0001 C CNN
+F 3 "~" H 3000 2950 50  0001 C CNN
+	1    3000 2950
 	-1   0    0    1
 $EndComp
@@
 L Device:C_Small C2
 U 1 1 5B84734E
-P 3850 3100
-F 0 "C2" H 3758 3054 50  0000 R CNN
-F 1 "22p" H 3758 3145 50  0000 R CNN
-F 2 "Capacitor_SMD:C_0805_2012Metric_Pad1.15x1.40mm_HandSolder" H 3850 3100 50  0001 C CNN
-F 3 "~" H 3850 3100 50  0001 C CNN
-	1    3850 3100
+P 3850 2950
+F 0 "C2" H 3758 2904 50  0000 R CNN
+F 1 "22p" H 3758 2995 50  0000 R CNN
+F 2 "Capacitor_SMD:C_0805_2012Metric_Pad1.15x1.40mm_HandSolder" H 3850 2950 50  0001 C CNN
+F 3 "~" H 3850 2950 50  0001 C CNN
+	1    3850 2950
 	-1   0    0    1
 $EndComp
-$Comp
-L Smallpaw-rescue:XTAL_GND-keyboard_parts X1
-U 1 1 5B847427
-P 3450 2900
-F 0 "X1" H 3450 3192 60  0000 C CNN
-F 1 "XTAL_GND" H 3450 3086 60  0000 C CNN
-F 2 "keyboard_parts:FA-238" H 3450 2900 60  0001 C CNN
-F 3 "" H 3450 2900 60  0000 C CNN
-	1    3450 2900
-	1    0    0    -1
-$EndComp
-Wire Wire Line
-	3000 2900 3150 2900
-Wire Wire Line
-	3000 2650 3000 2900
-Wire Wire Line
-	3750 2900 3850 2900
-Wire Wire Line
-	3000 3250 3450 3250
-Wire Wire Line
-	3450 3250 3450 3100
-Wire Wire Line
-	3850 3250 3450 3250
-Connection ~ 3450 3250
-Wire Wire Line
-	3450 3400 3450 3250
-Wire Wire Line
-	3000 2900 3000 3000
-Connection ~ 3000 2900
-Wire Wire Line
-	3000 3200 3000 3250
-Wire Wire Line
-	3850 2900 3850 3000
-Wire Wire Line
-	3850 3200 3850 3250
 $Comp
 L power:GND #PWR0101
 U 1 1 5B847D3A
-P 3450 3400
-F 0 "#PWR0101" H 3450 3150 50  0001 C CNN
-F 1 "GND" H 3455 3227 50  0000 C CNN
-F 2 "" H 3450 3400 50  0001 C CNN
-F 3 "" H 3450 3400 50  0001 C CNN
-	1    3450 3400
-	1    0    0    -1
-$EndComp
-Wire Wire Line
-	3000 2650 4400 2650
+P 3450 3050
+F 0 "#PWR0101" H 3450 2800 50  0001 C CNN
+F 1 "GND" H 3455 2877 50  0000 C CNN
+F 2 "" H 3450 3050 50  0001 C CNN
+F 3 "" H 3450 3050 50  0001 C CNN
+	1    3450 3050
+	1    0    0    -1
+$EndComp
+Wire Wire Line
+	3000 2650 3450 2650
 Wire Wire Line
 	4400 2750 3850 2750
 Wire Wire Line
-	3850 2750 3850 2900
-Connection ~ 3850 2900
-$Comp
-L power:VCC #PWR0102
-U 1 1 5B847F99
-P 1600 950
-F 0 "#PWR0102" H 1600 800 50  0001 C CNN
-F 1 "VCC" H 1617 1123 50  0000 C CNN
-F 2 "" H 1600 950 50  0001 C CNN
-F 3 "" H 1600 950 50  0001 C CNN
-	1    1600 950
-	1    0    0    -1
-$EndComp
+	3850 2750 3850 2850
 $Comp
 L power:GND #PWR0103
@@
 Wire Wire Line
 	1600 950  1600 1050
-Connection ~ 1600 950
 $Comp
 L Smallpaw-rescue:SW_PUSH-keyboard_parts SW1
@@
 F 0 "SW1" H 3650 2605 50  0000 C CNN
 F 1 "SW_PUSH" H 3650 2514 50  0000 C CNN
-F 2 "Button_Switch_SMD:SW_SPST_TL3342" H 3650 2350 60  0001 C CNN
+F 2 "Buttons_Switches_SMD:SW_SPST_SKQG" H 3650 2350 60  0001 C CNN
 F 3 "" H 3650 2350 60  0000 C CNN
 	1    3650 2350
 	1    0    0    -1
-$EndComp
-$Comp
-L power:VCC #PWR0104
-U 1 1 5B84D7E3
-P 3250 2150
-F 0 "#PWR0104" H 3250 2000 50  0001 C CNN
-F 1 "VCC" V 3268 2277 50  0000 L CNN
-F 2 "" H 3250 2150 50  0001 C CNN
-F 3 "" H 3250 2150 50  0001 C CNN
-	1    3250 2150
-	0    -1   -1   0
 $EndComp
 $Comp
@@
 F 0 "J1" H 3436 1691 60  0000 C CNN
 F 1 "USB_mini_micro_B" H 3400 1650 60  0001 C CNN
-F 2 "keyboard_parts:USB_microB" H 3500 1400 60  0001 C CNN
+F 2 "keebio-parts:USB-Mini-B_ LCSC-C46398" H 3500 1400 60  0001 C CNN
 F 3 "" H 3500 1400 60  0000 C CNN
 	1    3550 1400
 	1    0    0    -1
 $EndComp
-Wire Wire Line
-	3700 1250 3850 1250
 $Comp
 L power:VCC #PWR0107
 U 1 1 5B8543DB
-P 3850 1150
-F 0 "#PWR0107" H 3850 1000 50  0001 C CNN
-F 1 "VCC" H 3867 1323 50  0000 C CNN
-F 2 "" H 3850 1150 50  0001 C CNN
-F 3 "" H 3850 1150 50  0001 C CNN
-	1    3850 1150
-	1    0    0    -1
-$EndComp
-Wire Wire Line
-	3850 1150 3850 1250
-Connection ~ 3850 1250
-Wire Wire Line
-	3850 1250 4400 1250
+P 3800 1250
+F 0 "#PWR0107" H 3800 1100 50  0001 C CNN
+F 1 "VCC" H 3817 1423 50  0000 C CNN
+F 2 "" H 3800 1250 50  0001 C CNN
+F 3 "" H 3800 1250 50  0001 C CNN
+	1    3800 1250
+	1    0    0    -1
+$EndComp
 $Comp
 L Device:R R3
@@
 	3950 1550 4000 1550
 Connection ~ 4000 1550
-$Comp
-L power:VCC #PWR0109
-U 1 1 5B85D533
-P 4100 2450
-F 0 "#PWR0109" H 4100 2300 50  0001 C CNN
-F 1 "VCC" V 4118 2577 50  0000 L CNN
-F 2 "" H 4100 2450 50  0001 C CNN
-F 3 "" H 4100 2450 50  0001 C CNN
-	1    4100 2450
-	0    -1   -1   0
-$EndComp
 Wire Wire Line
 	4100 2450 4400 2450
-$Comp
-L power:VCC #PWR0110
-U 1 1 5B85F164
-P 4150 1750
-F 0 "#PWR0110" H 4150 1600 50  0001 C CNN
-F 1 "VCC" V 4168 1877 50  0000 L CNN
-F 2 "" H 4150 1750 50  0001 C CNN
-F 3 "" H 4150 1750 50  0001 C CNN
-	1    4150 1750
-	0    -1   -1   0
-$EndComp
 Wire Wire Line
 	4150 1750 4400 1750
@@
 Wire Wire Line
 	6650 3250 6550 3250
-$Comp
-L power:VCC #PWR0113
-U 1 1 5B86211E
-P 6750 3150
-F 0 "#PWR0113" H 6750 3000 50  0001 C CNN
-F 1 "VCC" V 6767 3278 50  0000 L CNN
-F 2 "" H 6750 3150 50  0001 C CNN
-F 3 "" H 6750 3150 50  0001 C CNN
-	1    6750 3150
-	0    1    1    0
-$EndComp
 Wire Wire Line
 	6750 3150 6550 3150
-$Comp
-L power:VCC #PWR0114
-U 1 1 5B863205
-P 6700 2150
-F 0 "#PWR0114" H 6700 2000 50  0001 C CNN
-F 1 "VCC" V 6717 2278 50  0000 L CNN
-F 2 "" H 6700 2150 50  0001 C CNN
-F 3 "" H 6700 2150 50  0001 C CNN
-	1    6700 2150
-	0    1    1    0
-$EndComp
 Wire Wire Line
 	6700 2150 6550 2150
@@
 Wire Wire Line
 	6700 1250 6550 1250
-$Comp
-L power:VCC #PWR0117
-U 1 1 5B86669E
-P 6650 1150
-F 0 "#PWR0117" H 6650 1000 50  0001 C CNN
-F 1 "VCC" V 6667 1278 50  0000 L CNN
-F 2 "" H 6650 1150 50  0001 C CNN
-F 3 "" H 6650 1150 50  0001 C CNN
-	1    6650 1150
-	0    1    1    0
-$EndComp
 Wire Wire Line
 	6650 1150 6550 1150
@@
 C7
 NoConn ~ 12750 4850
+Wire Wire Line
+	3700 1250 3800 1250
+$Comp
+L Device:Polyfuse_Small F1
+U 1 1 5E7E1EC6
+P 4050 1250
+F 0 "F1" V 3845 1250 50  0000 C CNN
+F 1 "500 mA" V 3936 1250 50  0000 C CNN
+F 2 "keebio-parts:Fuse_0805" H 4100 1050 50  0001 L CNN
+F 3 "~" H 4050 1250 50  0001 C CNN
+	1    4050 1250
+	0    1    1    0
+$EndComp
+Wire Wire Line
+	4150 1250 4300 1250
+Wire Wire Line
+	3950 1250 3800 1250
+Connection ~ 3800 1250
+$Comp
+L power:+5V #PWR0118
+U 1 1 5E831CCE
+P 4300 1250
+F 0 "#PWR0118" H 4300 1100 50  0001 C CNN
+F 1 "+5V" H 4315 1423 50  0000 C CNN
+F 2 "" H 4300 1250 50  0001 C CNN
+F 3 "" H 4300 1250 50  0001 C CNN
+	1    4300 1250
+	1    0    0    -1
+$EndComp
+Connection ~ 4300 1250
+Wire Wire Line
+	4300 1250 4400 1250
+$Comp
+L power:+5V #PWR0102
+U 1 1 5E84EF66
+P 1600 950
+F 0 "#PWR0102" H 1600 800 50  0001 C CNN
+F 1 "+5V" H 1615 1123 50  0000 C CNN
+F 2 "" H 1600 950 50  0001 C CNN
+F 3 "" H 1600 950 50  0001 C CNN
+	1    1600 950
+	1    0    0    -1
+$EndComp
+Connection ~ 1600 950
+$Comp
+L Device:Crystal_GND24_Small Y1
+U 1 1 5E86728D
+P 3450 2750
+F 0 "Y1" V 3404 2919 50  0000 L CNN
+F 1 "Crystal_GND24_Small" V 3495 2919 50  0000 L CNN
+F 2 "Crystals:Crystal_SMD_SeikoEpson_FA238-4pin_3.2x2.5mm" H 3450 2750 50  0001 C CNN
+F 3 "~" H 3450 2750 50  0001 C CNN
+	1    3450 2750
+	0    1    1    0
+$EndComp
+Connection ~ 3450 2650
+Wire Wire Line
+	3450 2650 4400 2650
+Wire Wire Line
+	3000 2650 3000 2850
+$Comp
+L power:+5V #PWR0109
+U 1 1 5E93B9B3
+P 6650 1150
+F 0 "#PWR0109" H 6650 1000 50  0001 C CNN
+F 1 "+5V" H 6665 1323 50  0000 C CNN
+F 2 "" H 6650 1150 50  0001 C CNN
+F 3 "" H 6650 1150 50  0001 C CNN
+	1    6650 1150
+	1    0    0    -1
+$EndComp
+$Comp
+L power:+5V #PWR0113
+U 1 1 5E93C185
+P 6750 3150
+F 0 "#PWR0113" H 6750 3000 50  0001 C CNN
+F 1 "+5V" H 6765 3323 50  0000 C CNN
+F 2 "" H 6750 3150 50  0001 C CNN
+F 3 "" H 6750 3150 50  0001 C CNN
+	1    6750 3150
+	1    0    0    -1
+$EndComp
+$Comp
+L power:+5V #PWR0114
+U 1 1 5E993EB9
+P 6700 2150
+F 0 "#PWR0114" H 6700 2000 50  0001 C CNN
+F 1 "+5V" V 6715 2278 50  0000 L CNN
+F 2 "" H 6700 2150 50  0001 C CNN
+F 3 "" H 6700 2150 50  0001 C CNN
+	1    6700 2150
+	0    1    1    0
+$EndComp
+$Comp
+L power:+5V #PWR0117
+U 1 1 5E9B1DE1
+P 4100 2450
+F 0 "#PWR0117" H 4100 2300 50  0001 C CNN
+F 1 "+5V" V 4115 2578 50  0000 L CNN
+F 2 "" H 4100 2450 50  0001 C CNN
+F 3 "" H 4100 2450 50  0001 C CNN
+	1    4100 2450
+	0    -1   -1   0
+$EndComp
+Wire Wire Line
+	3325 2750 3325 3050
+Connection ~ 3850 2850
+Wire Wire Line
+	3850 2850 3450 2850
+Wire Wire Line
+	3850 3050 3575 3050
+Connection ~ 3325 3050
+Wire Wire Line
+	3000 3050 3325 3050
+Wire Wire Line
+	3575 2750 3575 3050
+Wire Wire Line
+	3450 3050 3325 3050
+Wire Wire Line
+	3450 3050 3575 3050
+Connection ~ 3450 3050
+Connection ~ 3575 3050
+$Comp
+L power:+5V #PWR0110
+U 1 1 5ED1826F
+P 4150 1750
+F 0 "#PWR0110" H 4150 1600 50  0001 C CNN
+F 1 "+5V" V 4165 1878 50  0000 L CNN
+F 2 "" H 4150 1750 50  0001 C CNN
+F 3 "" H 4150 1750 50  0001 C CNN
+	1    4150 1750
+	0    -1   -1   0
+$EndComp
+$Comp
+L power:+5V #PWR?
+U 1 1 5ED3AA84
+P 3250 2150
+F 0 "#PWR?" H 3250 2000 50  0001 C CNN
+F 1 "+5V" H 3265 2323 50  0000 C CNN
+F 2 "" H 3250 2150 50  0001 C CNN
+F 3 "" H 3250 2150 50  0001 C CNN
+	1    3250 2150
+	1    0    0    -1
+$EndComp
 $EndSCHEMATC
